Commit message: switch to Gazebo native control and fix physics

File: src/gazebo_harmonic/urdf/hunter_base.xacro (robot description, xacro)
@@ -85,5 +85,5 @@
     <plugin filename="gz-sim-imu-system" name="gz::sim::systems::Imu"/>
     <plugin filename="gz-sim-navsat-system" name="gz::sim::systems::NavSat"/>
-    <plugin filename="gz-sim-wheel-slip-system" name="gz::sim::systems::WheelSlip">
+    <!-- <plugin filename="gz-sim-wheel-slip-system" name="gz::sim::systems::WheelSlip">
       <wheel link_name="rear_left_link">
         <slip_compliance_lateral>0.0</slip_compliance_lateral>
@@ -110,5 +110,5 @@
         <wheel_normal_force>171.5</wheel_normal_force>
       </wheel>
-    </plugin>
+    </plugin> -->
 </gazebo>
 <!-- <gazebo reference="imu_link">
@@ -128,12 +128,12 @@
     <imu>
       <angular_velocity>
-        <x><noise type="gaussian"><mean>0</mean><stddev>0.001</stddev></noise></x>
-        <y><noise type="gaussian"><mean>0</mean><stddev>0.001</stddev></noise></y>
-        <z><noise type="gaussian"><mean>0</mean><stddev>0.001</stddev></noise></z>
+        <x><noise type="gaussian"><mean>0</mean><stddev>0.0</stddev></noise></x>
+        <y><noise type="gaussian"><mean>0</mean><stddev>0.0</stddev></noise></y>
+        <z><noise type="gaussian"><mean>0</mean><stddev>0.0</stddev></noise></z>
       </angular_velocity>
       <linear_acceleration>
-        <x><noise type="gaussian"><mean>0</mean><stddev>0.01</stddev></noise></x>
-        <y><noise type="gaussian"><mean>0</mean><stddev>0.01</stddev></noise></y>
-        <z><noise type="gaussian"><mean>0</mean><stddev>0.01</stddev></noise></z>
+        <x><noise type="gaussian"><mean>0</mean><stddev>0.0</stddev></noise></x>
+        <y><noise type="gaussian"><mean>0</mean><stddev>0.0</stddev></noise></y>
+        <z><noise type="gaussian"><mean>0</mean><stddev>0.0</stddev></noise></z>
       </linear_acceleration>
     </imu>

File: src/gazebo_harmonic/urdf/hunter_gazebo.xacro (robot description, xacro)
@@ -3,5 +3,5 @@
     <!-- Include Gazebo plugins -->
     <xacro:include filename="$(find gazebo_harmonic)/urdf/hunter_base.xacro"/>
-    <xacro:include filename="$(find gazebo_harmonic)/urdf/ros2_control.xacro"/>
+    <xacro:include filename="$(find gazebo_harmonic)/urdf/gazebo_control.xacro"/>
     <xacro:include filename="$(find gazebo_harmonic)/urdf/velodyne_VLP32C_gazebo.xacro"/>
     <!-- Include modular components -->

File: src/hunter_base/urdf/front_wheels.xacro (robot description, xacro)
@@ -31,5 +31,5 @@
     <axis xyz="0 1 0"/>
     <limit lower="-0.576" upper="0.576" effort="1000" velocity="1000"/>
-    <dynamics damping="0.7"/>
+    <dynamics damping="0.2"/>
   </joint>
   <link name="front_left_wheel_link">
@@ -52,5 +52,6 @@
       <origin xyz="0 0 0" rpy="0 0 0"/>
       <geometry>
-        <cylinder radius="0.165" length="0.14"/>
+        <!-- Reduced length to 0.01 to prevent steering interference with chassis -->
+        <cylinder radius="0.165" length="0.01"/>
       </geometry>
     </collision>
@@ -61,5 +62,5 @@
     <child link="front_left_wheel_link"/>
     <axis xyz="0 0 -1"/>
-    <dynamics damping="0.7"/>
+    <dynamics damping="0.2"/>
   </joint>
   <!-- ========== Front Right Steering Link & Wheel ========== -->
@@ -93,5 +94,5 @@
     <axis xyz="0 1 0"/>
     <limit lower="-0.576" upper="0.576" effort="1000" velocity="1000"/>
-    <dynamics damping="0.7"/>
+    <dynamics damping="0.2"/>
   </joint>
   <link name="front_right_wheel_link">
@@ -114,5 +115,6 @@
       <origin xyz="0 0 0" rpy="0 0 0"/>
       <geometry>
-        <cylinder radius="0.165" length="0.14"/>
+        <!-- Reduced length to 0.01 to prevent steering interference with chassis -->
+        <cylinder radius="0.165" length="0.01"/>
       </geometry>
     </collision>
@@ -123,5 +125,5 @@
     <child link="front_right_wheel_link"/>
     <axis xyz="0 0 -1"/>
-    <dynamics damping="0.7"/>
+    <dynamics damping="0.2"/>
   </joint>
 </robot>

File: src/hunter_base/urdf/rear_wheels.xacro (robot description, xacro)
@@ -30,5 +30,5 @@
     <axis xyz="0 0 -1"/>
     <limit effort="10" velocity="100"/>
-    <dynamics damping="0.7"/>
+    <dynamics damping="0.2"/>
   </joint>
   <link name="rear_right_link">
@@ -61,5 +61,5 @@
     <axis xyz="0 0 -1"/>
     <limit effort="10" velocity="100"/>
-    <dynamics damping="0.7"/>
+    <dynamics damping="0.2"/>
   </joint>
 </robot>
