Commit message: fix tf tree and xacro

File: src/gazebo_harmonic/urdf/gazebo_control.xacro (robot description, xacro)
@@ -10,5 +10,5 @@
       <right_steering_joint>front_steer_right_joint</right_steering_joint>
       <kingpin_width>0.585</kingpin_width>
-      <steering_limit>0.576</steering_limit>
+      <steering_limit>0.461</steering_limit>
       <wheel_base>0.65142</wheel_base>
       <wheel_separation>0.585</wheel_separation>
@@ -20,8 +20,8 @@
       <topic>/cmd_vel</topic>
       <odom_topic>/odom</odom_topic>
-      <tf_topic>/tf</tf_topic>
+      <odom_publish_frequency>50</odom_publish_frequency>
       <frame_id>odom</frame_id>
       <child_frame_id>base_link</child_frame_id>
-      <odom_publish_frequency>50</odom_publish_frequency>
+      <tf_topic>/tf_gz</tf_topic>
     </plugin>
     <plugin
@@ -35,6 +35,6 @@
       name="gz::sim::systems::OdometryPublisher">
       <odom_frame>world</odom_frame>
-      <robot_base_frame>base_link_gt</robot_base_frame>
-      <odom_topic>/ground_truth/odom</odom_topic>
+      <robot_base_frame>base_link_ground_truth</robot_base_frame>
+      <odom_topic>/odometry/ground_truth</odom_topic>
       <tf_topic>/tf</tf_topic>
       <dimensions>3</dimensions>

File: src/gazebo_harmonic/urdf/hunter_base.xacro (robot description, xacro)
@@ -85,39 +85,5 @@
     <plugin filename="gz-sim-imu-system" name="gz::sim::systems::Imu"/>
     <plugin filename="gz-sim-navsat-system" name="gz::sim::systems::NavSat"/>
-    <!-- <plugin filename="gz-sim-wheel-slip-system" name="gz::sim::systems::WheelSlip">
-      <wheel link_name="rear_left_link">
-        <slip_compliance_lateral>0.0</slip_compliance_lateral>
-        <slip_compliance_longitudinal>0.0</slip_compliance_longitudinal>
-        <wheel_radius>0.165</wheel_radius>
-        <wheel_normal_force>171.5</wheel_normal_force>
-      </wheel>
-      <wheel link_name="rear_right_link">
-        <slip_compliance_lateral>0.0</slip_compliance_lateral>
-        <slip_compliance_longitudinal>0.0</slip_compliance_longitudinal>
-        <wheel_radius>0.165</wheel_radius>
-        <wheel_normal_force>171.5</wheel_normal_force>
-      </wheel>
-      <wheel link_name="front_left_wheel_link">
-        <slip_compliance_lateral>0.0</slip_compliance_lateral>
-        <slip_compliance_longitudinal>0.0</slip_compliance_longitudinal>
-        <wheel_radius>0.165</wheel_radius>
-        <wheel_normal_force>171.5</wheel_normal_force>
-      </wheel>
-      <wheel link_name="front_right_wheel_link">
-        <slip_compliance_lateral>0.0</slip_compliance_lateral>
-        <slip_compliance_longitudinal>0.0</slip_compliance_longitudinal>
-        <wheel_radius>0.165</wheel_radius>
-        <wheel_normal_force>171.5</wheel_normal_force>
-      </wheel>
-    </plugin> -->
 </gazebo>
-<!-- <gazebo reference="imu_link">
-  <sensor name="imu_sensor" type="imu">
-    <always_on>true</always_on>
-    <update_rate>100</update_rate>
-    <visualize>true</visualize>
-    <topic>imu</topic>
-  </sensor>
-</gazebo> -->
 <gazebo reference="imu_link">
   <sensor name="imu_sensor" type="imu">
@@ -126,14 +92,15 @@
     <visualize>true</visualize>
     <topic>imu</topic>
+    <frame_id>imu_link</frame_id>
     <imu>
       <angular_velocity>
-        <x><noise type="gaussian"><mean>0</mean><stddev>0.0</stddev></noise></x>
-        <y><noise type="gaussian"><mean>0</mean><stddev>0.0</stddev></noise></y>
-        <z><noise type="gaussian"><mean>0</mean><stddev>0.0</stddev></noise></z>
+        <x><noise type="gaussian"><mean>0</mean><stddev>0.000001</stddev></noise></x>
+        <y><noise type="gaussian"><mean>0</mean><stddev>0.000001</stddev></noise></y>
+        <z><noise type="gaussian"><mean>0</mean><stddev>0.000001</stddev></noise></z>
       </angular_velocity>
       <linear_acceleration>
-        <x><noise type="gaussian"><mean>0</mean><stddev>0.0</stddev></noise></x>
-        <y><noise type="gaussian"><mean>0</mean><stddev>0.0</stddev></noise></y>
-        <z><noise type="gaussian"><mean>0</mean><stddev>0.0</stddev></noise></z>
+        <x><noise type="gaussian"><mean>0</mean><stddev>0.000001</stddev></noise></x>
+        <y><noise type="gaussian"><mean>0</mean><stddev>0.000001</stddev></noise></y>
+        <z><noise type="gaussian"><mean>0</mean><stddev>0.000001</stddev></noise></z>
       </linear_acceleration>
     </imu>
@@ -145,5 +112,12 @@
     <update_rate>10</update_rate>
     <topic>gps</topic>
-  </sensor>
+    <frame_id>gps_link</frame_id>
+    <navsat>
+      <position_sensing>
+        <horizontal><noise type="gaussian"><mean>0.0</mean><stddev>0.00001</stddev></noise></horizontal>
+        <vertical><noise type="gaussian"><mean>0.0</mean><stddev>0.00001</stddev></noise></vertical>
+      </position_sensing>
+    </navsat>
+    </sensor>
 </gazebo>
 </robot>

File: src/hunter_base/urdf/front_wheels.xacro (robot description, xacro)
@@ -30,5 +30,6 @@
     <child link="front_steer_left_link"/>
     <axis xyz="0 1 0"/>
-    <limit lower="-0.576" upper="0.576" effort="1000" velocity="1000"/>
+    <!-- <limit lower="-0.576" upper="0.576" effort="1000" velocity="1000"/> -->
+    <limit lower="-0.461" upper="0.461" effort="1000" velocity="1000"/>
     <dynamics damping="0.2"/>
   </joint>
@@ -93,5 +94,6 @@
     <child link="front_steer_right_link"/>
     <axis xyz="0 1 0"/>
-    <limit lower="-0.576" upper="0.576" effort="1000" velocity="1000"/>
+    <!-- <limit lower="-0.576" upper="0.576" effort="1000" velocity="1000"/> -->
+    <limit lower="-0.461" upper="0.461" effort="1000" velocity="1000"/>
     <dynamics damping="0.2"/>
   </joint>
