Commit message: Sync Harmonic with Fortress features and fix inconsistencies
- Add camera sensor (HD 1280x720, 15Hz, 120° FOV) on front_box
- Add vehicle_speed_publisher node (/odom -> /vehicle/speed)
- Fix baylands launch: restore full bridge (9 topics), static TFs, custom nodes
- Add for_rviz flag for conditional logo rendering in Gazebo/rviz2
- Switch spawn method to -string with xacro for_rviz control
- Sync hunter_base URDFs: colors, material names, collision origins, LiDAR height
- Fix velodyne mesh path (model:// -> file://), joint type (fixed -> revolute)
- Add physics config to empty_with_gps.sdf (1ms step)
- Update CMakeLists/package.xml with new dependencies
- Rewrite README with full documentation
- Update .gitignore

Co-Authored-By: Claude Opus 4.6 (1M context) <noreply@anthropic.com>

File: src/gazebo_harmonic/urdf/hunter_gazebo.xacro (robot description, xacro)
@@ -1,8 +1,11 @@
 <?xml version="1.0"?>
 <robot xmlns:xacro="http://www.ros.org/wiki/xacro"  name="hunter2">
+    <xacro:arg name="for_rviz" default="false"/>
+    <xacro:property name="for_rviz" value="$(arg for_rviz)"/>
     <!-- Include Gazebo plugins -->
     <xacro:include filename="$(find gazebo_harmonic)/urdf/hunter_base.xacro"/>
     <xacro:include filename="$(find gazebo_harmonic)/urdf/gazebo_control.xacro"/>
     <xacro:include filename="$(find gazebo_harmonic)/urdf/velodyne_VLP32C_gazebo.xacro"/>
+    <xacro:include filename="$(find gazebo_harmonic)/urdf/camera_gazebo.xacro"/>
     <!-- Include modular components -->
     <xacro:include filename="$(find hunter_base)/urdf/base_link.xacro"/>
@@ -12,3 +15,4 @@
     <xacro:include filename="$(find hunter_base)/urdf/rear_wheels.xacro"/>
     <xacro:include filename="$(find hunter_base)/urdf/velodyne_VLP32C.xacro"/>
+    <xacro:include filename="$(find hunter_base)/urdf/camera.xacro"/>
 </robot>

File: src/hunter_base/urdf/base_link.xacro (robot description, xacro)
@@ -25,6 +25,6 @@
         <mesh filename="file://$(find hunter_base)/meshes/base_link.stl"/>
       </geometry>
-      <material name="black">
-        <color rgba="0.1 0.1 0.1 1"/>
+      <material name="chassis_dark_gray">
+        <color rgba="0.3 0.3 0.3 1"/>
       </material>
     </visual>

File: src/hunter_base/urdf/front_box_link.xacro (robot description, xacro)
@@ -13,8 +13,9 @@
         <mesh filename="file://$(find hunter_base)/meshes/front_box_with_logo_only_body.stl" scale="0.01 0.01 0.01"/>
       </geometry>
-      <material name="white">
+      <material name="front_box_white">
         <color rgba="1.0 1.0 1.0 1.0"/>
       </material>
     </visual>
+    <xacro:unless value="${for_rviz}">
     <visual name="box_visual_logo">
       <origin xyz="0 0 0" rpy="0 0 0"/>
@@ -22,8 +23,9 @@
         <mesh filename="file://$(find hunter_base)/meshes/front_box_with_logo_only_logo.stl" scale="0.01 0.01 0.01"/>
       </geometry>
-      <material name="navy">
+      <material name="front_box_navy">
         <color rgba="0.0 0.0 0.5 1.0"/>
       </material>
     </visual>
+    </xacro:unless>
     <visual name="box_visual_shadow">
       <origin xyz="0 0 0" rpy="0 0 0"/>
@@ -31,10 +33,10 @@
         <mesh filename="file://$(find hunter_base)/meshes/front_box_with_logo_only_shadow.stl" scale="0.01 0.01 0.01"/>
       </geometry>
-      <material name="black">
-        <color rgba="0.1 0.1 0.1 1.0"/>
+      <material name="front_box_shadow">
+        <color rgba="0.15 0.15 0.15 1.0"/>
       </material>
     </visual>
     <collision>
-      <origin xyz="0 0 0" rpy="0 0 0"/>
+      <origin xyz="0.228 0.185 0.138" rpy="0 0 0"/>
       <geometry>
         <box size="0.455 0.370 0.275"/>

File: src/hunter_base/urdf/front_wheels.xacro (robot description, xacro)
@@ -15,5 +15,5 @@
       </geometry>
       <material name="">
-        <color rgba="0.79216 0.81961 0.93333 1"/>
+        <color rgba="0.3 0.3 0.3 1"/>
       </material>
     </visual>
@@ -47,5 +47,5 @@
       </geometry>
       <material name="">
-        <color rgba="0.79216 0.81961 0.93333 1"/>
+        <color rgba="0.3 0.3 0.3 1"/>
       </material>
     </visual>
@@ -79,5 +79,5 @@
       </geometry>
       <material name="">
-        <color rgba="0.79216 0.81961 0.93333 1"/>
+        <color rgba="0.3 0.3 0.3 1"/>
       </material>
     </visual>
@@ -111,5 +111,5 @@
       </geometry>
       <material name="">
-        <color rgba="0.79216 0.81961 0.93333 1"/>
+        <color rgba="0.3 0.3 0.3 1"/>
       </material>
     </visual>

File: src/hunter_base/urdf/rear_box_link.xacro (robot description, xacro)
@@ -13,8 +13,9 @@
         <mesh filename="file://$(find hunter_base)/meshes/rear_box_with_logo_body.stl" scale="0.001 0.001 0.001"/>
       </geometry>
-      <material name="white">
+      <material name="rear_box_white">
         <color rgba="1.0 1.0 1.0 1.0"/>
       </material>
     </visual>
+    <xacro:unless value="${for_rviz}">
     <visual name="rear_box_visual_logo">
       <origin xyz="0 0 0" rpy="0 0 0"/>
@@ -22,8 +23,9 @@
         <mesh filename="file://$(find hunter_base)/meshes/rear_box_with_logo_logo.stl" scale="0.001 0.001 0.001"/>
       </geometry>
-      <material name="navy">
+      <material name="rear_box_navy">
         <color rgba="0.0 0.0 0.5 1.0"/>
       </material>
     </visual>
+    </xacro:unless>
     <visual name="rear_box_visual_shadow">
       <origin xyz="0 0 0" rpy="0 0 0"/>
@@ -31,12 +33,12 @@
         <mesh filename="file://$(find hunter_base)/meshes/rear_box_with_logo_shadow.stl" scale="0.001 0.001 0.001"/>
       </geometry>
-      <material name="black">
-        <color rgba="0.1 0.1 0.1 1.0"/>
+      <material name="rear_box_shadow">
+        <color rgba="0.15 0.15 0.15 1.0"/>
       </material>
     </visual>
     <collision>
-      <origin xyz="0 0 0" rpy="0 0 0"/>
+      <origin xyz="0.180 0.250 0.083" rpy="0 0 0"/>
       <geometry>
-        <box size="0.455 0.370 0.275"/>
+        <box size="0.360 0.500 0.165"/>
       </geometry>
     </collision>

File: src/hunter_base/urdf/rear_wheels.xacro (robot description, xacro)
@@ -14,5 +14,5 @@
       </geometry>
       <material name="">
-        <color rgba="0.79216 0.81961 0.93333 1"/>
+        <color rgba="0.3 0.3 0.3 1"/>
       </material>
     </visual>
@@ -45,5 +45,5 @@
       </geometry>
       <material name="">
-        <color rgba="0.79216 0.81961 0.93333 1"/>
+        <color rgba="0.3 0.3 0.3 1"/>
       </material>
     </visual>

File: src/hunter_base/urdf/velodyne_VLP32C.xacro (robot description, xacro)
@@ -11,5 +11,5 @@
       <origin xyz="0 0 0" rpy="0 0 0"/>
       <geometry>
-        <mesh filename="model://Lidar 3d v1/meshes/lidar_3d_v1.dae"/>
+        <mesh filename="file://$(find hunter_base)/meshes/lidar_3d_v1.dae"/>
       </geometry>
     </visual>
@@ -27,8 +27,10 @@
     </inertial>
   </link>
-  <joint name="lidar_visual_joint" type="fixed">
+  <joint name="lidar_visual_joint" type="revolute">
     <parent link="front_box"/>
     <child link="lidar_visual_link"/>
-    <origin xyz="0.23 0.14 0.28" rpy="0 0 1.5708"/>
+    <origin xyz="0.23 0.14 0.30" rpy="0 0 1.5708"/>
+    <axis xyz="0 0 1"/>
+    <limit lower="0" upper="0" effort="0" velocity="0"/>
   </joint>
   <joint name="lidar_sensor_joint" type="fixed">
