Commit message: Replace with Gazebo Fortress (Ignition 6) simulation
Fortress branch: uses ignition-gazebo-* plugins, RGL GPU LiDAR,
and ignition.msgs.* bridge types for Gazebo Fortress (Ignition 6).

Co-Authored-By: Claude Opus 4.6 (1M context) <noreply@anthropic.com>

File: src/gazebo_fortress/urdf/gazebo_control.xacro (robot description, xacro)
@@ -3,6 +3,6 @@
   <gazebo>
     <plugin
-      filename="gz-sim-ackermann-steering-system"
-      name="gz::sim::systems::AckermannSteering">
+      filename="ignition-gazebo-ackermann-steering-system"
+      name="ignition::gazebo::systems::AckermannSteering">
       <left_joint>rear_left_joint</left_joint>
       <right_joint>rear_right_joint</right_joint>
@@ -19,23 +19,23 @@
       <max_acceleration>5</max_acceleration>
       <topic>/cmd_vel</topic>
-      <odom_topic>/odom</odom_topic>
+      <odom_topic>/odometry/wheel</odom_topic>
       <odom_publish_frequency>50</odom_publish_frequency>
       <frame_id>odom</frame_id>
       <child_frame_id>base_link</child_frame_id>
-      <tf_topic>/tf_gz</tf_topic>
+      <tf_topic>/tf_wheel</tf_topic>
     </plugin>
     <plugin
-        filename="gz-sim-joint-state-publisher-system"
-        name="gz::sim::systems::JointStatePublisher">
+        filename="ignition-gazebo-joint-state-publisher-system"
+        name="ignition::gazebo::systems::JointStatePublisher">
         <topic>joint_states</topic>
         <update_rate>50</update_rate>
     </plugin>
     <plugin
-      filename="gz-sim-odometry-publisher-system"
-      name="gz::sim::systems::OdometryPublisher">
+      filename="ignition-gazebo-odometry-publisher-system"
+      name="ignition::gazebo::systems::OdometryPublisher">
       <odom_frame>world</odom_frame>
       <robot_base_frame>base_link_ground_truth</robot_base_frame>
       <odom_topic>/odometry/ground_truth</odom_topic>
-      <tf_topic>/tf</tf_topic>
+      <tf_topic>/tf_gt</tf_topic>
       <dimensions>3</dimensions>
       <odom_publish_frequency>50</odom_publish_frequency>

File: src/gazebo_fortress/urdf/hunter_base.xacro (robot description, xacro)
@@ -83,6 +83,6 @@
 </gazebo>
 <gazebo>
-    <plugin filename="gz-sim-imu-system" name="gz::sim::systems::Imu"/>
-    <plugin filename="gz-sim-navsat-system" name="gz::sim::systems::NavSat"/>
+    <plugin filename="ignition-gazebo-imu-system" name="ignition::gazebo::systems::Imu"/>
+    <plugin filename="ignition-gazebo-navsat-system" name="ignition::gazebo::systems::NavSat"/>
 </gazebo>
 <gazebo reference="imu_link">
@@ -119,5 +119,5 @@
       </position_sensing>
     </navsat>
-    </sensor>
+  </sensor>
 </gazebo>
 </robot>

File: src/gazebo_fortress/urdf/hunter_gazebo.xacro (robot description, xacro)
@@ -4,8 +4,8 @@
     <xacro:property name="for_rviz" value="$(arg for_rviz)"/>
     <!-- Include Gazebo plugins -->
-    <xacro:include filename="$(find gazebo_harmonic)/urdf/hunter_base.xacro"/>
-    <xacro:include filename="$(find gazebo_harmonic)/urdf/gazebo_control.xacro"/>
-    <xacro:include filename="$(find gazebo_harmonic)/urdf/velodyne_VLP32C_gazebo.xacro"/>
-    <xacro:include filename="$(find gazebo_harmonic)/urdf/camera_gazebo.xacro"/>
+    <xacro:include filename="$(find gazebo_fortress)/urdf/hunter_base.xacro"/>
+    <xacro:include filename="$(find gazebo_fortress)/urdf/gazebo_control.xacro"/>
+    <xacro:include filename="$(find gazebo_fortress)/urdf/velodyne_VLP32C_gazebo.xacro"/>
+    <xacro:include filename="$(find gazebo_fortress)/urdf/camera_gazebo.xacro"/>
     <!-- Include modular components -->
     <xacro:include filename="$(find hunter_base)/urdf/base_link.xacro"/>

File: src/hunter_base/urdf/base_link.xacro (robot description, xacro)
@@ -25,5 +25,5 @@
         <mesh filename="file://$(find hunter_base)/meshes/base_link.stl"/>
       </geometry>
-      <material name="chassis_dark_gray">
+      <material name="black">
         <color rgba="0.3 0.3 0.3 1"/>
       </material>
